File: stm32f1.kicad_pcb (KiCad board)
At the start: 2 copper layers, 28 parts, among them J1 Conn_01x04_Pin, J2 USB_B_Micro, J3 Conn_01x04_Pin, J4 Conn_01x04_Pin, SW1 SW_SPDT, U1 STM32F103C8T6, U3 AMS1117-3.3, Y1 16GHz

Commit message: add pcb
Parts:
- added H1: MountingHole, MountingHole:MountingHole_2.2mm_M2, F.Cu at (104.9, 50.0)
- added H2: MountingHole, MountingHole:MountingHole_2.2mm_M2, F.Cu at (139.9, 50.0)
- added H3: MountingHole, MountingHole:MountingHole_2.2mm_M2, F.Cu at (139.9, 79.9)
- added H4: MountingHole, MountingHole:MountingHole_2.2mm_M2, F.Cu at (104.9, 79.9)
- C1: footprint Capacitor_SMD:C_0201_0603Metric -> Capacitor_SMD:C_0402_1005Metric
- SW1: footprint Button_Switch_THT:SW_E-Switch_EG1224_SPDT_Angled -> Button_Switch_SMD:SW_SPDT_PCM12
- moved J1 132.5 mm to (131.1, 48.6), turned to -90 degrees
- moved R3 132.3 mm to (140.6, 71.1), turned to 90 degrees
- moved J2 128.2 mm to (139.8, 61.9), turned to 90 degrees
- moved D1 126.5 mm to (140.6, 74.5), turned to -90 degrees
- moved J4 120.9 mm to (115.2, 81.2), turned to 90 degrees
- moved R2 120.3 mm to (130.6, 61.3), turned to -90 degrees
- moved U3 118.8 mm to (131.0, 73.7), turned to -90 degrees
- moved C13 116.9 mm to (136.3, 73.5), turned to 90 degrees
- moved J3 115.3 mm to (118.1, 48.6), turned to -90 degrees
- moved U1 115.2 mm to (120.3, 63.2)
- moved C5 114.5 mm to (123.4, 69.5), turned to 180 degrees
- moved SW1 114.2 mm to (103.7, 57.6), turned to -90 degrees
- moved C4 113.7 mm to (126.7, 60.8), turned to -90 degrees
- moved R5 112.2 mm to (119.6, 73.5)
- moved C12 111.7 mm to (131.9, 67.7)
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Routing:
- net +3.3V: track 0.00 -> 175.6 mm, vias 0 -> 4
- net GND: track 0.00 -> 40.7 mm, vias 0 -> 19
- net Net-(U1-BOOT0): track 0.00 -> 17.6 mm
- net /I2C2_SCL: track 0.00 -> 16.8 mm
- net /SWDIO: track 0.00 -> 16.1 mm
- net /USART1_RX: track 0.00 -> 15.8 mm
- net VBUS: track 0.00 -> 15.2 mm
- net /USART1_TX: track 0.00 -> 14.9 mm
- net /I2C2_SDA: track 0.00 -> 14.7 mm
- net /USB_D-: track 0.00 -> 13.4 mm
- net /USB_D+: track 0.00 -> 13.4 mm
- net /SWCLK: track 0.00 -> 11.7 mm
- net /NRST: track 0.00 -> 9.37 mm
- net /HSE_IN: track 0.00 -> 9.11 mm
- net +3.3VA: track 0.00 -> 8.65 mm
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- added copper zone on B.Cu, net GND
Other:
- board outline added: 42.5 x 37.3 mm
- board text added: "-"
- board text added: "ON"
- board text added: "RX"
- board text added: "SWCLK"
- board text added: "SWDIO"
- board text added: "TX"
